Commit message: fix on review #1

File: my_robot/urdf/my_robot.xacro (robot description, xacro)
@@ -13,4 +13,7 @@
   <gazebo reference="camera">
     <material>Gazebo/Green</material>
+  </gazebo>
+  <gazebo reference="hokuyo_stand">
+    <material>Gazebo/Black</material>
   </gazebo>
   <link name="robot_footprint"></link>
@@ -42,8 +45,14 @@
     <axis xyz="0 1 0" />
   </joint>
+  <joint type="fixed" name="hokuyo_stand_joint">
+    <origin xyz="0.36 0 0.1" rpy="0 0 0" />
+    <child link="hokuyo_stand" />
+    <parent link="chassis" />
+    <axis xyz="0 1 0" />
+  </joint>
   <joint type="fixed" name="hokuyo_joint">
-    <origin xyz="0.3 0 0.1" rpy="0 0 0" />
+    <origin xyz="0 0 0.1" rpy="0 0 0" />
     <child link="hokuyo" />
-    <parent link="chassis" />
+    <parent link="hokuyo_stand" />
     <axis xyz="0 1 0" />
   </joint>
@@ -74,5 +83,5 @@
       <origin xyz="-0.3 0 -0.1" rpy=" 0 0 0"/>
       <geometry>
-        <sphere radius="0.1"/>
+        <sphere radius="0.099"/>
       </geometry>
     </collision>
@@ -82,10 +91,9 @@
         <sphere radius="0.1"/>
       </geometry>
-      <material name="">Gazebo/Green</material>
     </visual>
     <collision name='front_caster_collision'>
       <origin xyz="0.3 0 -0.1" rpy=" 0 0 0"/>
       <geometry>
-        <sphere radius="0.1"/>
+        <sphere radius="0.099"/>
       </geometry>
     </collision>
@@ -95,5 +103,4 @@
         <sphere radius="0.1"/>
       </geometry>
-      <material name="">Gazebo/Green</material>
     </visual>
   </link>
@@ -119,5 +126,4 @@
         <cylinder radius="0.2" length="0.1" />
       </geometry>
-      <material name="">Gazebo/Blue</material>
     </visual>
   </link>
@@ -143,5 +149,4 @@
         <cylinder radius="0.2" length="0.1" />
       </geometry>
-      <material name="">Gazebo/Blue</material>
     </visual>
   </link>
@@ -191,3 +196,26 @@
     </visual>
   </link>
+  <link name="hokuyo_stand">
+    <inertial>
+      <mass value="0.1" />
+      <origin xyz="0 0 0" rpy="0 0 0" />
+      <box_inertia m="0.1" x="0.05" y="0.05" z="0.05"/>
+      <inertia
+          ixx="1e-6" ixy="0" ixz="0"
+          iyy="1e-6" iyz="0"
+          izz="1e-6" />
+    </inertial>
+    <collision>
+      <origin xyz="0 0 0" rpy="0 0 0" />
+      <geometry>
+        <box size="0.05 0.05 0.2" />
+      </geometry>
+    </collision>
+    <visual>
+      <origin xyz="0 0 0" rpy="0 0 0" />
+      <geometry>
+        <box size="0.05 0.05 0.15" />
+      </geometry>
+    </visual>
+  </link>
 </robot>
