Commit message: add optical camera link

File: catkin_ws/src/my_robot/urdf/my_robot.xacro (robot description, xacro)
@@ -57,4 +57,9 @@
     <axis xyz="0 1 0" />
   </joint>
+  <joint type="fixed" name="camera_optical_joint">
+    <origin xyz="0 0 0" rpy="-1.5707 0 -1.5707"/>
+    <parent link="camera"/>
+    <child link="camera_link_optical"/>
+  </joint>
   <link name='chassis'>
     <pose>0 0 0.2 0 0 0</pose>
@@ -219,3 +224,5 @@
     </visual>
   </link>
+  <link name="camera_link_optical">
+  </link>
 </robot>
